File: pcb/DaviShematic.sch (EAGLE design)
At the start: 11 parts, among them IC1 MEGA8-P, IC2 L293D

Commit message: Add files via upload
Parts:
- C1, C2: value (none) -> 1uF; device rcl:C-US025-024X044 -> rcl:C-EU025-025X050
- R1: value 10k -> (none); device rcl:R-US_0207/7 -> rcl:R-EU_0204/7
Connections:
- net GND: now also C1.1, C2.1; no longer C1.2, C2.2
- net N$2: now also C1.2; no longer C1.1
- net N$3: now also C2.2; no longer C2.1
Other:
- moved on the sheet: C1, C2
